File: WS2811_PWM_Driver.sch (KiCad schematic (older format))
At the start: 43 parts, among them P1 Com, P2 PWM, P3 HS/LS, P4 HS/LS, P5 GND, P6 DIFIN, P7 DIFOUT, Q1 AO3401, Q2 AO3401, Q3 AO3401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

Commit message: PCB Update
Parts:
- removed Q1, Q2, Q3, Q4, Q5, Q6: AO3401, TO_SOT_Packages_SMD:SOT-23, symbol AO3401
- removed R19, R20, R21, R22, R23, R24: 510, Resistors_SMD:R_0805, symbol R_SMD_0805
- added Q1, Q2, Q3, Q4, Q5, Q6: MMBT4401, WS2811_PWM_PCB:SOT-23, symbol Q_NPN_BEC
- R10, R12, R8: value 33 -> 510; footprint Resistors_SMD:R_0805 -> Resistors_SMD:R_0603
- R11, R7, R9: value 33 -> 4K7; footprint Resistors_SMD:R_0805 -> Resistors_SMD:R_0603
- R13, R15, R17: value 330 -> 4K7; footprint Resistors_SMD:R_0805 -> Resistors_SMD:R_0603
- R14, R16, R18: value 330 -> 510; footprint Resistors_SMD:R_0805 -> Resistors_SMD:R_0603

Commit message: PCB_Gerbers
Parts:
- added C3, C4: 10u/10V, Capacitors_SMD:C_0805, symbol C_Cer_SMD_0805
- R10, R12, R14, R16, R18, R8: value 510 -> 9.1K
Connections:
- wire segments 143 -> 153
Other:
- note added: "400KHz LOW SPEED Mode for very long wiring short jumpers P3, P4\nIf jumpers open 800KHz Default Mode"
- note added: "Long Wiring Differential In/Out:\nDifferential Drivers: U1/U2 \nTerminating Resistors: R1/R2\nJumpers P6/P7: Open"
- note added: "Operating in direct mode: \nU1,U2,R1,R2 - Not assembled\nP6,P7 Shorted"
- moved on the sheet: C1, C2, P1, P2, P3, P4, P5, P6, P7, Q1, Q2, Q3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
