File: WS2811_PWM_Driver.kicad_pcb (KiCad board)
At the start: 2 copper layers, 43 parts, among them P1 Com, P2 PWM, P3 HS/LS, P4 HS/LS, P5 GND, P6 DIFIN, P7 DIFOUT, Q1 AO3401, Q2 AO3401, Q3 AO3401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

Commit message: PCB Update
Parts:
- removed R19, R20, R21, R22, R23, R24: 510, Resistors_SMD:R_0805
- P3, P4, P5, P6, P7: moved to B.Cu
- Q1, Q2, Q3, Q4, Q5, Q6: value AO3401 -> MMBT4401; footprint PCB FootPrints:SOT-23 -> WS2811_PWM_PCB:SOT-23
- R10, R12, R8: value 33 -> 510; footprint Resistors_SMD:R_0805 -> Resistors_SMD:R_0603
- R11, R7, R9: value 33 -> 4K7; footprint Resistors_SMD:R_0805 -> Resistors_SMD:R_0603
- R13, R15, R17: value 330 -> 4K7; footprint Resistors_SMD:R_0805 -> Resistors_SMD:R_0603
- R14, R16, R18: value 330 -> 510; footprint Resistors_SMD:R_0805 -> Resistors_SMD:R_0603
- moved P6 94.2 mm to (106.1, 109.3), turned to 270 degrees
- moved P3 89.5 mm to (103.6, 122.8)
- moved R15 88.0 mm to (113.9, 105.7), turned to 270 degrees
- moved C2 87.8 mm to (104.6, 102.3), turned to 90 degrees
- moved R5 86.8 mm to (104.5, 107.8), turned to 90 degrees
- moved R13 84.5 mm to (113.9, 110.0), turned to 270 degrees
- moved R3 82.8 mm to (102.7, 122.9), turned to 270 degrees
- moved R7 78.4 mm to (113.9, 122.3), turned to 270 degrees
- moved R17 78.2 mm to (113.9, 102.2), turned to 270 degrees
- moved R4 77.1 mm to (102.7, 102.2), turned to 270 degrees
- moved R18 76.1 mm to (118.9, 101.9), turned to 270 degrees
- moved R12 75.9 mm to (118.9, 114.1), turned to 270 degrees
- moved C1 73.0 mm to (104.5, 122.7), turned to 90 degrees
- moved R14 70.2 mm to (119.0, 110.0), turned to 270 degrees
- moved Q5 70.0 mm to (116.4, 106.4)
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Connections:
- P1 pad 2: /INB -> /OUTB
- P1 pad 3: /INA -> /OUTA
- P1 pad 4: /OUTB -> /INB
- P1 pad 5: /OUTA -> /INA
- Q1 pad 1: Net-(Q1-Pad1) -> /Out1
- Q1 pad 2: +5V -> GND
- Q2 pad 1: Net-(Q2-Pad1) -> /Out2
- Q2 pad 2: +5V -> GND
- Q3 pad 1: Net-(Q3-Pad1) -> /Out3
- Q3 pad 2: +5V -> GND
- Q4 pad 1: Net-(Q4-Pad1) -> /Out4
- Q4 pad 2: +5V -> GND
- Q5 pad 1: Net-(Q5-Pad1) -> /Out5
- Q5 pad 2: +5V -> GND
- Q6 pad 1: Net-(Q6-Pad1) -> /Out6
- Q6 pad 2: +5V -> GND
- R10 pad 1: Net-(Q4-Pad1) -> +5V
- R10 pad 2: +5V -> /PWM2
- R11 pad 1: Net-(Q5-Pad1) -> +5V
- R11 pad 2: +5V -> /Out3
- R12 pad 1: Net-(Q6-Pad1) -> +5V
- R12 pad 2: +5V -> /PWM3
- R13 pad 1: /Out1 -> +5V
- R13 pad 2: Net-(Q1-Pad1) -> /Out4
- R14 pad 1: /Out2 -> +5V
- R14 pad 2: Net-(Q2-Pad1) -> /PWM4
- R15 pad 1: /Out3 -> +5V
- R15 pad 2: Net-(Q3-Pad1) -> /Out5
- R16 pad 1: /Out4 -> +5V
- R16 pad 2: Net-(Q4-Pad1) -> /PWM5
- R17 pad 1: /Out5 -> +5V
- R17 pad 2: Net-(Q5-Pad1) -> /Out6
- R18 pad 1: /Out6 -> +5V
- R18 pad 2: Net-(Q6-Pad1) -> /PWM6
- R7 pad 1: Net-(Q1-Pad1) -> +5V
- R7 pad 2: +5V -> /Out1
- R8 pad 1: Net-(Q2-Pad1) -> +5V
- R8 pad 2: +5V -> /PWM1
- R9 pad 1: Net-(Q3-Pad1) -> +5V
- R9 pad 2: +5V -> /Out2
- U1 pad 4: Net-(U1-Pad4) -> (no net)
- U4 pad 1: Net-(U4-Pad1) -> (no net)
Routing:
- net +5V: track 0.00 -> 98.2 mm, vias 0 -> 2
- net GND: track 0.00 -> 24.8 mm, vias 0 -> 14
- net Net-(R6-Pad1): track 0.00 -> 22.0 mm
- net /DI3: track 0.00 -> 21.6 mm, vias 0 -> 1
- net Net-(R5-Pad1): track 0.00 -> 20.1 mm, vias 0 -> 2
- net /DI1: track 0.00 -> 10.9 mm, vias 0 -> 2
- net /PWM1: track 0.00 -> 10.6 mm
- net /Out3: track 0.00 -> 9.32 mm
- net /PWM2: track 0.00 -> 9.09 mm
- net /INB: track 0.00 -> 9.03 mm, vias 0 -> 1
- net /PWM6: track 0.00 -> 8.49 mm
- net /OUTB: track 0.00 -> 8.12 mm, vias 0 -> 1
- net /Out4: track 0.00 -> 7.78 mm
- net /PWM5: track 0.00 -> 7.21 mm
- net /PWM3: track 0.00 -> 6.76 mm
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- added copper zone on B.Cu, net GND
Other:
- board outline added: 25 x 25 mm

Commit message: PCB_Gerbers
Parts:
- added C3: 10u/10V, Capacitors_SMD:C_0805, F.Cu at (120.5, 118.3)
- added C4: 10u/10V, Capacitors_SMD:C_0805, F.Cu at (120.6, 106.1)
- added REF***: KiCad-Logo2_6mm_SilkScreen, Symbols:KiCad-Logo2_6mm_SilkScreen, B.Cu at (115.4, 121.3)
- added REF***: OSHW-Logo_5.7x6mm_SilkScreen, Symbols:OSHW-Logo_5.7x6mm_SilkScreen, B.Cu at (119.1, 114.9)
Connections:
- P3 pad 1: GND -> +5V
- P4 pad 1: GND -> +5V
Routing:
- net +5V: track 98.2 -> 111.4 mm, vias 2 -> 4
- net GND: track 24.8 -> 28.0 mm, vias 14 -> 16
- net /PWM6: track 8.49 -> 10.0 mm
- net /PWM5: track 7.21 -> 8.32 mm
Other:
- board text added: "1"
- board text added: "5V"
- board text added: "6"
- board text added: "GND"
- board text added: "INA"
- board text added: "INB"
- board text added: "OUA"
- board text added: "OUB"
- board text added: "P3,P4-Open:HS Closed:LS"
- board text added: "P6,P7-Open:485 Closed:Direct"
- board text added: "PWM:400Hz/5V/5mA Power: 5V DC"
- board text added: "WS2811 6Ch PWM Driver V1.0 BK 2017"

Commit message: Gerber Updates
Parts:
- P3, P4, P6, P7: footprint mysensors_obscurities:2_pin_solder_jumper_smd -> BK_Common:2_pin_solder_jumper_smd
- moved REF*** 0.29 mm to (119.4, 115.0)
Changed lines of the file:
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@@
   (general
     (links 91)
-    (no_connects 2)
+    (no_connects 0)
     (area 99.924999 99.924999 125.075001 125.075001)
     (thickness 1.6)
@@
     )
   )
-  (module mysensors_obscurities:2_pin_solder_jumper_smd (layer B.Cu)
-    (at 103.632 122.7582)
-    (fp_text reference P3 (at 0 -1.5494 180) (layer B.SilkS)
-      (effects (font (size 0.75 0.75) (thickness 0.15)) (justify mirror))
-    )
-    (fp_text value HS/LS (at 0 1.524) (layer B.Fab)
-      (effects (font (size 1 1) (thickness 0.15)) (justify mirror))
-    )
-    (pad 2 smd oval (at 0.889 0) (size 1.27 1.524) (layers B.Cu B.Paste B.Mask)
-      (net 15 "Net-(P3-Pad2)"))
-    (pad 1 smd oval (at -0.889 0) (size 1.27 1.524) (layers B.Cu B.Paste B.Mask)
-      (net 4 +5V))
-  )
-  (module mysensors_obscurities:2_pin_solder_jumper_smd (layer B.Cu)
-    (at 103.6066 102.2604)
-    (fp_text reference P4 (at 0 1.651 180) (layer B.SilkS)
-      (effects (font (size 0.75 0.75) (thickness 0.15)) (justify mirror))
-    )
-    (fp_text value HS/LS (at 0 1.524) (layer B.Fab)
-      (effects (font (size 1 1) (thickness 0.15)) (justify mirror))
-    )
-    (pad 2 smd oval (at 0.889 0) (size 1.27 1.524) (layers B.Cu B.Paste B.Mask)
-      (net 16 "Net-(P4-Pad2)"))
-    (pad 1 smd oval (at -0.889 0) (size 1.27 1.524) (layers B.Cu B.Paste B.Mask)
-      (net 4 +5V))
-  )
   (module "PCB FootPrints:Pin_Header_Straight_1x06_Pitch2.00mm" (layer B.Cu)
     (at 123.3932 117.1758)
@@
       (rotate (xyz 0 0 0))
     )
-  )
-  (module mysensors_obscurities:2_pin_solder_jumper_smd (layer B.Cu)
-    (at 106.0704 109.3216 270)
-    (fp_text reference P6 (at -2.1844 0.1524 360) (layer B.SilkS)
-      (effects (font (size 0.75 0.75) (thickness 0.15)) (justify mirror))
-    )
-    (fp_text value DIFIN (at 0 1.524 270) (layer B.Fab)
-      (effects (font (size 1 1) (thickness 0.15)) (justify mirror))
-    )
-    (pad 2 smd oval (at 0.889 0 270) (size 1.27 1.524) (layers B.Cu B.Paste B.Mask)
-      (net 5 /INB))
-    (pad 1 smd oval (at -0.889 0 270) (size 1.27 1.524) (layers B.Cu B.Paste B.Mask)
-      (net 17 /DI1))
-  )
-  (module mysensors_obscurities:2_pin_solder_jumper_smd (layer B.Cu)
-    (at 106.1212 113.3348 270)
-    (fp_text reference P7 (at 2.3368 0 360) (layer B.SilkS)
-      (effects (font (size 0.75 0.75) (thickness 0.15)) (justify mirror))
-    )
-    (fp_text value DIFOUT (at 0 1.524 270) (layer B.Fab)
-      (effects (font (size 1 1) (thickness 0.15)) (justify mirror))
-    )
-    (pad 2 smd oval (at 0.889 0 270) (size 1.27 1.524) (layers B.Cu B.Paste B.Mask)
-      (net 7 /OUTB))
-    (pad 1 smd oval (at -0.889 0 270) (size 1.27 1.524) (layers B.Cu B.Paste B.Mask)
-      (net 18 /DI3))
   )
   (module Resistors_SMD:R_0805 (layer F.Cu)
@@
   )
   (module Symbols:OSHW-Logo_5.7x6mm_SilkScreen (layer B.Cu)
-    (at 119.126 114.9096 180)
+    (at 119.4 115 180)
     (descr "Open Source Hardware Logo")
     (tags "Logo OSHW")
@@
       (xy 0.376964 2.709982)) (layer B.SilkS) (width 0.01))
   )
+  (module BK_Common:2_pin_solder_jumper_smd (layer B.Cu)
+    (at 103.632 122.7582)
+    (fp_text reference P3 (at -2.1844 0.1524 90) (layer B.SilkS)
+      (effects (font (size 0.75 0.75) (thickness 0.15)) (justify mirror))
+    )
+    (fp_text value HS/LS (at 0 1.524) (layer B.Fab)
+      (effects (font (size 1 1) (thickness 0.15)) (justify mirror))
+    )
+    (fp_line (start 0 -0.9906) (end 0 1.0668) (layer B.Mask) (width 0.15))
+    (fp_line (start -0.1524 -1.016) (end -0.1524 1.0668) (layer B.Mask) (width 0.15))
+    (fp_line (start 0.127 -1.016) (end -0.1524 -1.016) (layer B.Mask) (width 0.15))
+    (fp_line (start 0.127 1.0668) (end 0.127 -1.016) (layer B.Mask) (width 0.15))
+    (fp_line (start -0.1524 1.0668) (end 0.127 1.0668) (layer B.Mask) (width 0.15))
+    (pad 2 smd trapezoid (at 0.8 0) (size 1.27 1.524) (rect_delta 0.6 0 ) (layers B.Cu B.Paste B.Mask)
+      (net 15 "Net-(P3-Pad2)"))
+    (pad 1 smd trapezoid (at -0.8 0) (size 1.27 1.524) (rect_delta -0.6 0 ) (layers B.Cu B.Paste B.Mask)
+      (net 4 +5V))
+  )
+  (module BK_Common:2_pin_solder_jumper_smd (layer B.Cu)
+    (at 103.6066 102.2604)
+    (fp_text reference P4 (at -2.1844 0.1524 90) (layer B.SilkS)
+      (effects (font (size 0.75 0.75) (thickness 0.15)) (justify mirror))
+    )
+    (fp_text value HS/LS (at 0 1.524) (layer B.Fab)
+      (effects (font (size 1 1) (thickness 0.15)) (justify mirror))
+    )
+    (fp_line (start 0 -0.9906) (end 0 1.0668) (layer B.Mask) (width 0.15))
+    (fp_line (start -0.1524 -1.016) (end -0.1524 1.0668) (layer B.Mask) (width 0.15))
+    (fp_line (start 0.127 -1.016) (end -0.1524 -1.016) (layer B.Mask) (width 0.15))
+    (fp_line (start 0.127 1.0668) (end 0.127 -1.016) (layer B.Mask) (width 0.15))
+    (fp_line (start -0.1524 1.0668) (end 0.127 1.0668) (layer B.Mask) (width 0.15))
+    (pad 2 smd trapezoid (at 0.8 0) (size 1.27 1.524) (rect_delta 0.6 0 ) (layers B.Cu B.Paste B.Mask)
+      (net 16 "Net-(P4-Pad2)"))
+    (pad 1 smd trapezoid (at -0.8 0) (size 1.27 1.524) (rect_delta -0.6 0 ) (layers B.Cu B.Paste B.Mask)
+      (net 4 +5V))
+  )
+  (module BK_Common:2_pin_solder_jumper_smd (layer B.Cu)
+    (at 106.0704 109.3216 270)
+    (fp_text reference P6 (at -2.1844 0.1524 360) (layer B.SilkS)
+      (effects (font (size 0.75 0.75) (thickness 0.15)) (justify mirror))
+    )
+    (fp_text value DIFIN (at 0 1.524 270) (layer B.Fab)
+      (effects (font (size 1 1) (thickness 0.15)) (justify mirror))
+    )
+    (fp_line (start 0 -0.9906) (end 0 1.0668) (layer B.Mask) (width 0.15))
+    (fp_line (start -0.1524 -1.016) (end -0.1524 1.0668) (layer B.Mask) (width 0.15))
+    (fp_line (start 0.127 -1.016) (end -0.1524 -1.016) (layer B.Mask) (width 0.15))
+    (fp_line (start 0.127 1.0668) (end 0.127 -1.016) (layer B.Mask) (width 0.15))
+    (fp_line (start -0.1524 1.0668) (end 0.127 1.0668) (layer B.Mask) (width 0.15))
+    (pad 2 smd trapezoid (at 0.8 0 270) (size 1.27 1.524) (rect_delta 0.6 0 ) (layers B.Cu B.Paste B.Mask)
+      (net 5 /INB))
+    (pad 1 smd trapezoid (at -0.8 0 270) (size 1.27 1.524) (rect_delta -0.6 0 ) (layers B.Cu B.Paste B.Mask)
+      (net 17 /DI1))
+  )
+  (module BK_Common:2_pin_solder_jumper_smd (layer B.Cu)
+    (at 106.1212 113.3348 270)
+    (fp_text reference P7 (at -2.1844 0.1524 360) (layer B.SilkS)
+      (effects (font (size 0.75 0.75) (thickness 0.15)) (justify mirror))
+    )
+    (fp_text value DIFOUT (at 0 1.524 270) (layer B.Fab)
+      (effects (font (size 1 1) (thickness 0.15)) (justify mirror))
+    )
+    (fp_line (start 0 -0.9906) (end 0 1.0668) (layer B.Mask) (width 0.15))
+    (fp_line (start -0.1524 -1.016) (end -0.1524 1.0668) (layer B.Mask) (width 0.15))
+    (fp_line (start 0.127 -1.016) (end -0.1524 -1.016) (layer B.Mask) (width 0.15))
+    (fp_line (start 0.127 1.0668) (end 0.127 -1.016) (layer B.Mask) (width 0.15))
+    (fp_line (start -0.1524 1.0668) (end 0.127 1.0668) (layer B.Mask) (width 0.15))
+    (pad 2 smd trapezoid (at 0.8 0 270) (size 1.27 1.524) (rect_delta 0.6 0 ) (layers B.Cu B.Paste B.Mask)
+      (net 7 /OUTB))
+    (pad 1 smd trapezoid (at -0.8 0 270) (size 1.27 1.524) (rect_delta -0.6 0 ) (layers B.Cu B.Paste B.Mask)
+      (net 18 /DI3))
+  )
   (gr_text 6 (at 121.793 107.2134) (layer F.SilkS)
     (effects (font (size 0.75 0.75) (thickness 0.15)))
@@
     (effects (font (size 1 1) (thickness 0.2)) (justify mirror))
   )
-  (gr_text "WS2811 6Ch\nPWM Driver\nV1.0 \nBK 2017" (at 111.7854 115.189) (layer B.SilkS)
+  (gr_text "WS2811 6Ch\nPWM Driver\nV1.0 \nBK 2017" (at 112.4 115.189) (layer B.SilkS)
     (effects (font (size 1 1) (thickness 0.2)) (justify mirror))
   )
@@
     (effects (font (size 1 1) (thickness 0.2)) (justify mirror))
   )
-  (gr_text "P6,P7-Open:485\nClosed:Direct" (at 115.3414 108.839 360) (layer B.SilkS)
+  (gr_text "P6,P7-Open:485\nClosed:Direct" (at 115.3414 108.839) (layer B.SilkS)
     (effects (font (size 1 1) (thickness 0.2)) (justify mirror))
   )
